File: test/files/blink1_v1a.brd (EAGLE design)
At the start: 20.7 x 11.7 mm, 17 parts, among them IC1 TODSTUFF_ATTINY45TSSOP8

Commit message: updated simple example files to use special characters (µ)
Parts:
- C2: value 10uF -> 10µF
Changed lines of the file:
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@@
 <attribute name="NAME" x="14.6304" y="11.0998" size="0.381" layer="25" font="vector" ratio="10" rot="R270"/>
 </element>
-<element name="C2" library="rcl" package="C0603" value="10uF" x="14.732" y="8.128" smashed="yes" rot="R90">
+<element name="C2" library="rcl" package="C0603" value="10µF" x="14.732" y="8.128" smashed="yes" rot="R90">
 <attribute name="NAME" x="14.4526" y="7.8994" size="0.381" layer="25" font="vector" ratio="10"/>
 </element>
