File: test/files/blink1_v1a.sch (EAGLE design)
At the start: 17 parts, among them IC1 TODSTUFF_ATTINY45TSSOP8

Commit message: updated simple example files to use special characters (µ)
Parts:
- C2: value 10uF -> 10µF
Changed lines of the file:
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@@
 <part name="R1" library="rcl" deviceset="R-US_" device="R0402" value="68"/>
 <part name="R2" library="rcl" deviceset="R-US_" device="R0402" value="68"/>
-<part name="C2" library="rcl" deviceset="C-US" device="C0603" value="10uF"/>
+<part name="C2" library="rcl" deviceset="C-US" device="C0603" value="10µF"/>
 <part name="R3" library="rcl" deviceset="R-US_" device="R0402" value="1k5"/>
 <part name="P+2" library="supply1" deviceset="VCC" device=""/>
